File: Eagle files/Leah board.brd (EAGLE design)
At the start: 25.4 x 37.3 mm, 2 parts

Commit message: Board Tweaks
Other:
- board size 25.4 x 37.3 mm -> 25.4 x 33.7 mm
- board text removed: "#13"
- board text removed: "16 MHz"
- board text removed: "A7"
- board text removed: "BLK"
- board text removed: "FTDI Header"
- board text removed: "GND"
- board text removed: "GRN"
- board text removed: "Pro"
- board text removed: "Trinket!"
- board text removed: "pwr"
Changed lines of the file:
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@@
 <layer number="15" name="Route15" color="4" fill="6" visible="no" active="yes"/>
 <layer number="16" name="Bottom" color="1" fill="1" visible="yes" active="yes"/>
-<layer number="17" name="Pads" color="2" fill="1" visible="no" active="yes"/>
+<layer number="17" name="Pads" color="2" fill="1" visible="yes" active="yes"/>
 <layer number="18" name="Vias" color="2" fill="1" visible="yes" active="yes"/>
 <layer number="19" name="Unrouted" color="6" fill="1" visible="yes" active="yes"/>
@@
 <board>
 <plain>
-<wire x1="12.7" y1="0.4445" x2="12.7" y2="36.068" width="0" layer="20"/>
+<wire x1="12.7" y1="2.413" x2="12.7" y2="36.068" width="0" layer="20"/>
 <wire x1="12.7" y1="36.068" x2="-12.7" y2="36.068" width="0" layer="20"/>
-<wire x1="-12.7" y1="36.068" x2="-12.7" y2="0" width="0" layer="20"/>
-<wire x1="-12.7" y1="0" x2="-7.747" y2="0" width="0" layer="20"/>
-<wire x1="-7.747" y1="0" x2="-6.477" y2="-1.27" width="0" layer="20"/>
-<wire x1="-6.477" y1="-1.27" x2="2.7305" y2="-1.27" width="0" layer="20"/>
-<wire x1="2.7305" y1="-1.27" x2="4.0005" y2="0" width="0" layer="20"/>
-<wire x1="4.0005" y1="0" x2="8.509" y2="0" width="0" layer="20"/>
-<wire x1="8.509" y1="0" x2="12.7" y2="0.4445" width="0" layer="20"/>
+<wire x1="-12.7" y1="36.068" x2="-12.7" y2="2.413" width="0" layer="20"/>
+<wire x1="-12.7" y1="2.413" x2="12.7" y2="2.413" width="0" layer="20"/>
 <text x="6.0325" y="30.4165" size="1.016" layer="21" font="vector" ratio="10" rot="R270" align="center-right">BAT</text>
 <text x="6.1214" y="29.8069" size="1.016" layer="21" font="vector" ratio="10" rot="R90" align="center-right">G</text>
@@
 <text x="6.6675" y="8.89" size="1.016" layer="21" font="vector" ratio="10" align="center-right">TX</text>
 <text x="6.731" y="6.35" size="1.016" layer="21" font="vector" ratio="10" align="center-right">RX</text>
-<text x="-8.128" y="2.921" size="1.016" layer="21" font="vector" ratio="10" rot="R90" align="center-right">BLK</text>
-<text x="8.001" y="2.921" size="1.016" layer="21" font="vector" ratio="10" rot="R90" align="center-right">GRN</text>
 <text x="5.969" y="5.461" size="1.016" layer="21" font="vector" ratio="10" rot="R90" align="center-right">RST</text>
-<text x="4.699" y="2.794" size="1.016" layer="21" font="vector" ratio="10" align="center-right">TX</text>
-<text x="2.286" y="2.794" size="1.016" layer="21" font="vector" ratio="10" align="center-right">RX</text>
-<text x="-0.254" y="2.794" size="1.016" layer="21" font="vector" ratio="10" align="center-right">5V</text>
-<text x="-3.683" y="2.794" size="1.016" layer="21" font="vector" ratio="10" align="center-right">GND</text>
 <text x="-6.477" y="3.937" size="1.016" layer="21" font="vector" ratio="10" rot="R180" align="center-right">A5</text>
 <text x="-6.477" y="6.35" size="1.016" layer="21" font="vector" ratio="10" rot="R180" align="center-right">A4</text>
 <text x="-6.477" y="8.89" size="1.016" layer="21" font="vector" ratio="10" rot="R180" align="center-right">A3</text>
 <text x="-6.477" y="10.668" size="1.016" layer="21" font="vector" ratio="10" rot="R180" align="center-right">A2</text>
-<text x="-3.429" y="13.208" size="1.016" layer="21" font="vector" ratio="10" rot="R270" align="center-right">A7</text>
 <text x="-6.985" y="12.7" size="0.9652" layer="21" font="vector" ratio="10" rot="R180" align="center-right">A1</text>
 <text x="-7.112" y="15.367" size="0.889" layer="21" font="vector" ratio="10" rot="R180" align="center-right">A0</text>
@@
 <text x="-5.588" y="27.178" size="1.016" layer="21" font="vector" ratio="10" align="center-right">~</text>
 <text x="6.604" y="33.147" size="1.016" layer="21" font="vector" ratio="10" align="center-right">+</text>
-<text x="0.508" y="17.526" size="1.143" layer="21" font="vector" ratio="12" rot="R180" align="center">Trinket!</text>
-<text x="1.905" y="9.144" size="1.27" layer="21" font="vector" ratio="10" rot="R180" align="center-right">5V</text>
-<wire x1="1.397" y1="10.287" x2="1.397" y2="8.128" width="0.254" layer="21"/>
-<wire x1="1.397" y1="8.128" x2="4.445" y2="8.128" width="0.254" layer="21"/>
-<wire x1="4.445" y1="8.128" x2="4.445" y2="10.287" width="0.254" layer="21"/>
-<wire x1="4.445" y1="10.287" x2="1.397" y2="10.287" width="0.254" layer="21"/>
 <text x="-5.588" y="31.75" size="1.016" layer="21" font="vector" ratio="10" align="center-right">9</text>
 <text x="-5.588" y="32.258" size="1.016" layer="21" font="vector" ratio="10" align="center-right">~</text>
-<text x="-1.651" y="-0.508" size="1.016" layer="21" font="vector" ratio="12" align="center">FTDI Header</text>
-<text x="4.191" y="12.319" size="1.016" layer="21" font="vector" ratio="12" rot="R180" align="center">16
-MHz</text>
-<text x="0.127" y="18.796" size="1.27" layer="21" font="vector" ratio="12" rot="R180" align="center">Pro</text>
-<text x="1.524" y="27.559" size="1.016" layer="21" font="vector" ratio="12">pwr</text>
-<text x="-3.048" y="27.178" size="1.016" layer="21" font="vector" ratio="12">#13</text>
 </plain>
 <attributes>
@@
 <contactref element="JP1" pad="2"/>
 <polygon width="0.3048" layer="16">
-<vertex x="-12.7" y="36.83"/>
-<vertex x="-12.7" y="0"/>
-<vertex x="12.7" y="0"/>
-<vertex x="12.7" y="36.83"/>
+<vertex x="-12.7" y="36.068"/>
+<vertex x="-12.7" y="2.413"/>
+<vertex x="12.7" y="2.413"/>
+<vertex x="12.7" y="36.068"/>
 </polygon>
 </signal>
@@
 </board>
 </drawing>
-<compatibility>
-<note version="6.3" minversion="6.2.2" severity="warning">
-Since Version 6.2.2 text objects can contain more than one line,
-which will not be processed correctly with this version.
-</note>
-</compatibility>
 </eagle>

Commit message: Board work
Parts:
- added CONT_LED, INT_LED, LASER, POWER, PWR_LED: (no value), adafruit:JST-PH-2-SMT-RA
- added POT: (no value), adafruit:JSTPH3
- added X_SERVO, Y_SERVO: (no value), adafruit:1X03
- moved JP4 22.2 mm to (14.6, 17.9)
- moved JP1 22.2 mm to (29.8, 17.9)
Connections:
- removed net VBAT: JP1.1
- new net VCC: JP1.1, POWER.1
- net A2: now also POT.2
- net GND: now also LASER.2, POWER.2
Other:
- board size 25.4 x 33.7 mm -> 41.9 x 41.1 mm

Commit message: Board tweaks
Other:
- board size 41.9 x 41.1 mm -> 43.2 x 43.2 mm
Changed lines of the file:
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@@
 <board>
 <plain>
-<wire x1="41.91" y1="2.032" x2="41.91" y2="43.18" width="0" layer="20"/>
-<wire x1="41.91" y1="43.18" x2="2.032" y2="43.18" width="0" layer="20"/>
-<wire x1="2.032" y1="43.18" x2="2.032" y2="22.225" width="0" layer="20"/>
-<wire x1="2.032" y1="22.225" x2="0" y2="20.32" width="0" layer="20"/>
-<wire x1="0" y1="20.32" x2="0" y2="15.24" width="0" layer="20"/>
-<wire x1="0" y1="15.24" x2="2.032" y2="13.335" width="0" layer="20"/>
-<wire x1="2.032" y1="13.335" x2="2.032" y2="2.032" width="0" layer="20"/>
-<wire x1="2.032" y1="2.032" x2="41.91" y2="2.032" width="0" layer="20"/>
+<wire x1="43.18" y1="43.18" x2="0" y2="43.18" width="0" layer="20"/>
+<wire x1="0" y1="43.18" x2="0" y2="0" width="0" layer="20"/>
+<wire x1="0" y1="0" x2="43.18" y2="0" width="0" layer="20"/>
 <text x="28.2575" y="30.5435" size="1.016" layer="21" font="vector" ratio="10" rot="R270" align="center-right">BAT</text>
 <text x="28.3464" y="29.9339" size="1.016" layer="21" font="vector" ratio="10" rot="R90" align="center-right">G</text>
@@
 <text x="16.637" y="31.877" size="1.016" layer="21" font="vector" ratio="10" align="center-right">9</text>
 <text x="16.637" y="32.385" size="1.016" layer="21" font="vector" ratio="10" align="center-right">~</text>
-<hole x="1.651" y="17.78" drill="2.2"/>
-<hole x="21.717" y="20.955" drill="2.2"/>
+<hole x="1.524" y="3.81" drill="2.2"/>
+<hole x="1.524" y="41.402" drill="2.2"/>
+<hole x="40.132" y="4.064" drill="2.2"/>
+<hole x="39.878" y="41.275" drill="2.2"/>
 </plain>
 <attributes>
@@
 <contactref element="JP1" pad="2"/>
 <polygon width="0.3048" layer="16">
-<vertex x="2.032" y="43.18"/>
-<vertex x="2.032" y="22.225"/>
-<vertex x="0" y="20.32"/>
-<vertex x="0" y="15.24"/>
-<vertex x="2.032" y="13.335"/>
-<vertex x="2.032" y="2.032"/>
-<vertex x="41.91" y="2.032"/>
-<vertex x="41.91" y="43.18"/>
+<vertex x="0" y="43.18"/>
+<vertex x="0" y="0"/>
+<vertex x="43.18" y="0"/>
+<vertex x="43.18" y="43.18"/>
 </polygon>
 <contactref element="POWER" pad="2"/>

Commit message: Modification for present.
Parts:
- added CONT_MOS, INT_MOS, LASER_MOS, PWR_MOS, X_MOS, Y_MOS: 200mA/50V, SparkFun-DiscreteSemi:SOT23-3
- added R1, R2, R3, R4, R5, R6: 10K, SparkFun-Resistors:0603-RES
- moved POWER 32.3 mm to (21.7, 5.21), turned to 180 degrees
- moved JP1 9.06 mm to (29.0, 26.9)
- moved JP4 9.06 mm to (13.7, 26.9)
- moved CONT_LED 4.66 mm to (36.7, 33.1)
- moved X_SERVO 3.43 mm to (36.1, 11.2)
Connections:
- new net CONT_PWR: CONT_LED.1, CONT_MOS.2, R2.2
- new net INT_PWR: INT_LED.1, INT_MOS.2, R1.2
- new net LASER_PIN: LASER_MOS.1
- new net N$2: INT_MOS.1
- new net N$3: CONT_MOS.1
- new net N$4: PWR_MOS.1
- new net N$5: LASER_MOS.2, R4.2
- new net N$6: R6.2, Y_MOS.2, Y_SERVO.2
- new net N$7: R5.2, X_MOS.2, X_SERVO.2
- new net PLED_PWR: PWR_LED.1, PWR_MOS.2, R3.2
- new net XSERVO_PWR_PIN: X_MOS.1
- new net YSERVO_PWR_PIN: Y_MOS.1
- net A0: now also X_SERVO.3
- net A1: now also Y_SERVO.1
- net GND: now also CONT_LED.2, INT_LED.2, POT.3, PWR_LED.2, R1.1, R2.1, R3.1, R4.1, R5.1, R6.1, X_SERVO.1, Y_SERVO.3
- net VCC: now also CONT_MOS.3, INT_MOS.3, LASER_MOS.3, POT.1, PWR_MOS.3, X_MOS.3, Y_MOS.3
Other:
- board text added: "B R Y"

Commit message: Added base Event class and timer class
Timer and Task classes are now derived from Event class
Parts:
- moved R2 2.22 mm to (19.2, 24.5)
- moved X_SERVO 1.52 mm to (36.1, 12.7), turned to 180 degrees
- moved Y_SERVO 0.13 mm to (36.1, 19.1)
Other:
- board text added: "Y R B"
- board text removed: "B R Y"
Changed lines of the file:
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@@
 <hole x="40.132" y="4.064" drill="2.2"/>
 <hole x="39.878" y="41.275" drill="2.2"/>
-<text x="32.258" y="15.113" size="1.778" layer="25">B R Y</text>
+<text x="36.068" y="15.875" size="1.778" layer="25" align="center">Y R B</text>
 </plain>
 <attributes>
@@
 <element name="CONT_LED" library="adafruit" package="JST-PH-2-SMT-RA" value="" x="36.703" y="33.147"/>
 <element name="INT_LED" library="adafruit" package="JST-PH-2-SMT-RA" value="" x="6.477" y="7.874" rot="R90"/>
-<element name="X_SERVO" library="adafruit" package="1X03" value="" x="36.068" y="11.176"/>
-<element name="Y_SERVO" library="adafruit" package="1X03" value="" x="36.068" y="18.923"/>
+<element name="X_SERVO" library="adafruit" package="1X03" value="" x="36.068" y="12.7" rot="R180"/>
+<element name="Y_SERVO" library="adafruit" package="1X03" value="" x="36.068" y="19.05"/>
 <element name="LASER" library="adafruit" package="JST-PH-2-SMT-RA" value="" x="6.477" y="38.227" rot="R90"/>
 <element name="PWR_MOS" library="SparkFun-DiscreteSemi" package="SOT23-3" value="200mA/50V" x="22.352" y="15.621" rot="MR0">
@@
 <attribute name="PROD_ID" value="RES-00824" x="22.225" y="36.195" size="1.778" layer="28" rot="MR0" display="off"/>
 </element>
-<element name="R2" library="SparkFun-Resistors" package="0603-RES" value="10K" x="20.066" y="22.479" rot="MR0">
-<attribute name="PROD_ID" value="RES-00824" x="20.066" y="22.479" size="1.778" layer="28" rot="MR0" display="off"/>
+<element name="R2" library="SparkFun-Resistors" package="0603-RES" value="10K" x="19.177" y="24.511" rot="MR0">
+<attribute name="PROD_ID" value="RES-00824" x="19.177" y="24.511" size="1.778" layer="28" rot="MR0" display="off"/>
 </element>
 <element name="R3" library="SparkFun-Resistors" package="0603-RES" value="10K" x="24.384" y="12.954" rot="MR0">
@@
 <wire x1="40.64" y1="24.042" x2="35.703" y2="29.447" width="0" layer="19" extent="1-16"/>
 <wire x1="22.717" y1="8.907" x2="25.234" y2="12.954" width="0" layer="19" extent="1-16"/>
-<wire x1="10.193" y1="20.415" x2="20.916" y2="22.479" width="0" layer="19" extent="1-16"/>
-<wire x1="10.05" y1="27.956" x2="10.193" y2="20.415" width="0" layer="19" extent="1-1"/>
+<wire x1="10.05" y1="27.956" x2="20.027" y2="24.511" width="0" layer="19" extent="1-16"/>
+<wire x1="10.193" y1="20.415" x2="10.05" y2="27.956" width="0" layer="19" extent="1-1"/>
 <wire x1="10.177" y1="37.227" x2="10.05" y2="27.956" width="0" layer="19" extent="1-1"/>
 <wire x1="10.177" y1="6.874" x2="22.717" y2="8.907" width="0" layer="19" extent="1-1"/>
@@
 <contactref element="JP4" pad="7"/>
 <contactref element="X_SERVO" pad="3"/>
-<wire x1="13.716" y1="25.654" x2="38.608" y2="11.176" width="0" layer="19" extent="1-1"/>
+<wire x1="13.716" y1="25.654" x2="33.528" y2="12.7" width="0" layer="19" extent="1-1"/>
 </signal>
 <signal name="A1">
 <contactref element="JP4" pad="8"/>
 <contactref element="Y_SERVO" pad="1"/>
-<wire x1="13.716" y1="23.114" x2="33.528" y2="18.923" width="0" layer="19" extent="1-1"/>
+<wire x1="13.716" y1="23.114" x2="33.528" y2="19.05" width="0" layer="19" extent="1-1"/>
 </signal>
 <signal name="A2">
@@
 <contactref element="R5" pad="2"/>
 <contactref element="X_SERVO" pad="2"/>
-<wire x1="33.721" y1="4.588" x2="36.068" y2="11.176" width="0" layer="19" extent="16-16"/>
+<wire x1="33.721" y1="4.588" x2="36.068" y2="12.7" width="0" layer="19" extent="16-16"/>
 <wire x1="37.426" y1="2.667" x2="33.721" y2="4.588" width="0" layer="19" extent="16-16"/>
 </signal>
@@
 <contactref element="Y_SERVO" pad="2"/>
 <wire x1="36.891" y1="25.13" x2="40.64" y2="25.742" width="0" layer="19" extent="16-16"/>
-<wire x1="36.068" y1="18.923" x2="36.891" y2="25.13" width="0" layer="19" extent="16-16"/>
+<wire x1="36.068" y1="19.05" x2="36.891" y2="25.13" width="0" layer="19" extent="16-16"/>
 </signal>
 <signal name="INT_PWR">
@@
 <contactref element="R2" pad="2"/>
 <wire x1="21.148" y1="19.32" x2="37.703" y2="29.447" width="0" layer="19" extent="1-16"/>
-<wire x1="19.216" y1="22.479" x2="21.148" y2="19.32" width="0" layer="19" extent="16-16"/>
+<wire x1="18.327" y1="24.511" x2="21.148" y2="19.32" width="0" layer="19" extent="16-16"/>
 </signal>
 <signal name="PLED_PWR">
