File: Eagle files/Leah board.brd (EAGLE design)
At the start: 43.2 x 43.2 mm, 25 parts

Commit message: Tweaks
Parts:
- moved R3 6.07 mm to (37.0, 40.6), turned to 0 degrees
- moved LASER_MOS 1.97 mm to (10.7, 38.1)
- moved R4 1.26 mm to (6.10, 41.1), turned to 0 degrees
- moved POT 1.02 mm to (11.4, 4.95)
- moved Y_MOS 0.89 mm to (8.76, 12.8)
- moved LASER 0.63 mm to (4.32, 33.3)
- moved CONT_LED 0.51 mm to (37.8, 22.7)
- moved R2 0.46 mm to (35.6, 29.0)
- moved X_MOS 0.40 mm to (7.62, 20.6)
- moved R8 0.25 mm to (39.5, 29.0)
Routing:
- net VCC: track 121.7 -> 114.9 mm
- net PLED_PWR: track 8.76 -> 13.9 mm
- net D9: track 2.65 -> 3.89 mm
- net LASER_PWR: track 10.6 -> 11.7 mm
- net A4: track 6.07 -> 5.43 mm

Commit message: Tweaks
Parts:
- removed CONT_LED: (no value), adafruit:JST-PH-2-SMT-RA
- removed CONT_MOS: 200mA/50V, SparkFun-DiscreteSemi:SOT23-3
- added C1: 100uF, SparkFun-Capacitors:EIA7343
- added R10: 39, SparkFun-Resistors:0603-RES
- added SLEEP_MOS: 200mA/50V, SparkFun-DiscreteSemi:SOT23-3
- added SLP_LED: (no value), adafruit:JST-PH-2-SMT-RA
- X_MOS, Y_MOS: value 200mA/50V -> 2.6A/20V
- moved INT_LED 12.1 mm to (37.8, 22.7)
- moved INT_MOS 8.88 mm to (34.0, 16.8), turned to 180 degrees
- moved R4 0.92 mm to (5.21, 40.9), turned to 90 degrees
- renumbered PWR_LED to RUN_LED, PWR_MOS to RUN_MOS
Connections:
- net A0 renamed X_PWM_PIN
- net A1 renamed Y_PWM_PIN
- net A2 renamed POT_IN
- net A3 renamed X_PWR_PIN
- net A4 renamed Y_PWR_PIN
- net D8 renamed RUN_LED_PIN
- net D9 renamed LASER_PIN
- net PLED_PWR renamed RUN_LED_PWR
- removed net CONT_PWR: CONT_LED.1, CONT_MOS.2, R2.2
- removed net D3: INT_MOS.1, JP1.9
- removed net D4: CONT_MOS.1, JP1.8
- removed net INT_PWR: INT_LED.1, INT_MOS.2, R1.2
- removed net VCC: CONT_MOS.3, INT_MOS.3, JP1.4, LASER_MOS.3, POT.1, POWER.1, RUN_MOS.3, X_MOS.3, Y_MOS.3
- new net 5V: JP1.4, POT.1
- new net INT_LED_PIN: INT_MOS.1, JP1.8
- new net INT_LED_PWR: INT_LED.1, INT_MOS.2, R2.2
- new net N$1: C1.A, LASER.1, R10.1
- new net SLP_LED_PIN: JP1.9, SLEEP_MOS.1
- new net SLP_LED_PWR: R1.2, SLEEP_MOS.2, SLP_LED.1
- net GND: now also C1.C
- net LASER_PWR: now also R10.2; no longer LASER.1
- net N$10: now also SLP_LED.2; no longer INT_LED.2
- net N$9: now also INT_LED.2; no longer CONT_LED.2
- net VBAT: now also INT_MOS.3, LASER_MOS.3, POWER.1, RUN_MOS.3, SLEEP_MOS.3, X_MOS.3, Y_MOS.3
Routing:
- net VBAT: track 0.00 -> 127.6 mm, vias 0 -> 2
- net VCC: track 114.9 -> 0.00 mm, vias 2 -> 0
- net 5V: track 0.00 -> 34.2 mm, vias 0 -> 1
- net INT_LED_PWR: track 0.00 -> 16.6 mm
- net CONT_PWR: track 16.6 -> 0.00 mm
- net N$1: track 0.00 -> 16.2 mm, vias 0 -> 1
- net INT_LED_PIN: track 0.00 -> 11.8 mm
- net D4: track 11.8 -> 0.00 mm
- net SLP_LED_PIN: track 0.00 -> 11.3 mm
- net D3: track 11.3 -> 0.00 mm
- net SLP_LED_PWR: track 0.00 -> 11.2 mm
- net INT_PWR: track 11.2 -> 0.00 mm
- net LASER_PWR: track 11.7 -> 7.05 mm
- net GND: track 98.0 -> 96.0 mm
Other:
- board text removed: "From: Mom"
- board text removed: "To: Leah"
- board text removed: "XMAS 2014"
